File: encoderBreakout/encoderBreakout.kicad_pcb (KiCad board)
At the start: 2 copper layers, 32 x 31 mm, 2 parts, among them J1 Conn_01x08_MountingPin

Commit message: gitignore
Parts:
- moved encoderWithKailh1 50.6 mm to (150.5, 100.0)
- moved J1 7.64 mm to (141.4, 74.0), turned to 90 degrees
Other:
- board size 32 x 31 mm -> 49.5 x 51.5 mm
Changed lines of the file:
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@@
 	(footprint "Connector_PinSocket_2.54mm:PinSocket_1x08_P2.54mm_Vertical"
 		(layer "F.Cu")
-		(at 148.295 70.795)
+		(at 141.36 74 90)
 		(descr "Through hole straight socket strip, 1x08, 2.54mm pitch, single row (from Kicad 4.0.7), script generated")
 		(tags "Through hole socket strip THT 1x08 2.54mm single row")
 		(property "Reference" "J1"
-			(at 0 -2.77 0)
+			(at 0 -2.77 90)
 			(layer "F.SilkS")
 			(effects
@@
 		)
 		(property "Value" "Conn_01x08_MountingPin"
-			(at 0 20.55 0)
+			(at 0 20.55 90)
 			(layer "F.Fab")
 			(effects
@@
 		)
 		(property "Datasheet" ""
-			(at 0 0 0)
+			(at 0 0 90)
 			(layer "F.Fab")
 			(hide yes)
@@
 		)
 		(property "Description" "Generic connectable mounting pin connector, single row, 01x08, script generated (kicad-library-utils/schlib/autogen/connector/)"
-			(at 0 0 0)
+			(at 0 0 90)
 			(layer "F.Fab")
 			(hide yes)
@@
 		)
 		(property "KiLib_Generator" "connector/pin_header_socket"
-			(at 0 0 0)
+			(at 0 0 90)
 			(layer "F.SilkS")
 			(hide yes)
@@
 		(duplicate_pad_numbers_are_jumpers no)
 		(fp_line
+			(start 1.33 -1.33)
+			(end 1.33 0)
+			(stroke
+				(width 0.12)
+				(type solid)
+			)
+			(layer "F.SilkS")
+		)
+		(fp_line
+			(start 0 -1.33)
+			(end 1.33 -1.33)
+			(stroke
+				(width 0.12)
+				(type solid)
+			)
+			(layer "F.SilkS")
+		)
+		(fp_line
+			(start 1.33 1.27)
+			(end 1.33 19.11)
+			(stroke
+				(width 0.12)
+				(type solid)
+			)
+			(layer "F.SilkS")
+		)
+		(fp_line
+			(start -1.33 1.27)
+			(end 1.33 1.27)
+			(stroke
+				(width 0.12)
+				(type solid)
+			)
+			(layer "F.SilkS")
+		)
+		(fp_line
 			(start -1.33 1.27)
 			(end -1.33 19.11)
@@
 		)
 		(fp_line
-			(start -1.33 1.27)
-			(end 1.33 1.27)
-			(stroke
-				(width 0.12)
-				(type solid)
-			)
-			(layer "F.SilkS")
-		)
-		(fp_line
 			(start -1.33 19.11)
 			(end 1.33 19.11)
@@
 		)
 		(fp_line
-			(start 0 -1.33)
-			(end 1.33 -1.33)
-			(stroke
-				(width 0.12)
-				(type solid)
-			)
-			(layer "F.SilkS")
-		)
-		(fp_line
-			(start 1.33 -1.33)
-			(end 1.33 0)
-			(stroke
-				(width 0.12)
-				(type solid)
-			)
-			(layer "F.SilkS")
-		)
-		(fp_line
-			(start 1.33 1.27)
-			(end 1.33 19.11)
-			(stroke
-				(width 0.12)
-				(type solid)
-			)
-			(layer "F.SilkS")
+			(start 1.77 -1.77)
+			(end 1.77 19.55)
+			(stroke
+				(width 0.05)
+				(type solid)
+			)
+			(layer "F.CrtYd")
 		)
 		(fp_line
@@
 		)
 		(fp_line
+			(start 1.77 19.55)
+			(end -1.77 19.55)
+			(stroke
+				(width 0.05)
+				(type solid)
+			)
+			(layer "F.CrtYd")
+		)
+		(fp_line
 			(start -1.77 19.55)
 			(end -1.77 -1.77)
@@
 		)
 		(fp_line
-			(start 1.77 -1.77)
-			(end 1.77 19.55)
-			(stroke
-				(width 0.05)
-				(type solid)
-			)
-			(layer "F.CrtYd")
-		)
-		(fp_line
-			(start 1.77 19.55)
-			(end -1.77 19.55)
-			(stroke
-				(width 0.05)
-				(type solid)
-			)
-			(layer "F.CrtYd")
+			(start 0.635 -1.27)
+			(end 1.27 -0.635)
+			(stroke
+				(width 0.1)
+				(type solid)
+			)
+			(layer "F.Fab")
 		)
 		(fp_line
@@
 		)
 		(fp_line
+			(start 1.27 -0.635)
+			(end 1.27 19.05)
+			(stroke
+				(width 0.1)
+				(type solid)
+			)
+			(layer "F.Fab")
+		)
+		(fp_line
+			(start 1.27 19.05)
+			(end -1.27 19.05)
+			(stroke
+				(width 0.1)
+				(type solid)
+			)
+			(layer "F.Fab")
+		)
+		(fp_line
 			(start -1.27 19.05)
 			(end -1.27 -1.27)
@@
 			(layer "F.Fab")
 		)
-		(fp_line
-			(start 0.635 -1.27)
-			(end 1.27 -0.635)
-			(stroke
-				(width 0.1)
-				(type solid)
-			)
-			(layer "F.Fab")
-		)
-		(fp_line
-			(start 1.27 -0.635)
-			(end 1.27 19.05)
-			(stroke
-				(width 0.1)
-				(type solid)
-			)
-			(layer "F.Fab")
-		)
-		(fp_line
-			(start 1.27 19.05)
-			(end -1.27 19.05)
-			(stroke
-				(width 0.1)
-				(type solid)
-			)
-			(layer "F.Fab")
-		)
 		(fp_text user "${REFERENCE}"
-			(at 0 8.89 90)
+			(at 1 8.64 0)
 			(layer "F.Fab")
 			(effects
@@
 		)
 		(pad "1" thru_hole rect
-			(at 0 0)
+			(at 0 0 90)
 			(size 1.7 1.7)
 			(drill 1)
@@
 		)
 		(pad "2" thru_hole circle
-			(at 0 2.54)
+			(at 0 2.54 90)
 			(size 1.7 1.7)
 			(drill 1)
@@
 		)
 		(pad "3" thru_hole circle
-			(at 0 5.08)
+			(at 0 5.08 90)
 			(size 1.7 1.7)
 			(drill 1)
@@
 		)
 		(pad "4" thru_hole circle
-			(at 0 7.62)
+			(at 0 7.62 90)
 			(size 1.7 1.7)
 			(drill 1)
@@
 		)
 		(pad "5" thru_hole circle
-			(at 0 10.16)
+			(at 0 10.16 90)
 			(size 1.7 1.7)
 			(drill 1)
@@
 		)
 		(pad "6" thru_hole circle
-			(at 0 12.7)
+			(at 0 12.7 90)
 			(size 1.7 1.7)
 			(drill 1)
@@
 		)
 		(pad "7" thru_hole circle
-			(at 0 15.24)
+			(at 0 15.24 90)
 			(size 1.7 1.7)
 			(drill 1)
@@
 		)
 		(pad "8" thru_hole circle
-			(at 0 17.78)
+			(at 0 17.78 90)
 			(size 1.7 1.7)
 			(drill 1)
@@
 	(footprint "encLibrary:EC35AwithKailhSocket"
 		(layer "F.Cu")
-		(at 104.25 79.5)
+		(at 150.5 100)
 		(descr "35mm Size Ring Type")
 		(tags "encoder, rotary encoder")
@@
 			(polygon
 				(pts
-					(xy 102.35 85.9) (xy 106.15 85.9) (xy 106.15 82.5) (xy 102.35 82.5)
+					(xy 148.6 106.4) (xy 152.4 106.4) (xy 152.4 103) (xy 148.6 103)
 				)
 			)
@@
 			(polygon
 				(pts
-					(xy 102.35 85.9) (xy 106.15 85.9) (xy 106.15 82.5) (xy 102.35 82.5)
+					(xy 148.6 106.4) (xy 152.4 106.4) (xy 152.4 103) (xy 148.6 103)
 				)
 			)
@@
 		)
 	)
+	(gr_rect
+		(start 125.5 70)
+		(end 175 121.5)
+		(stroke
+			(width 0.05)
+			(type default)
+		)
+		(fill no)
+		(layer "Edge.Cuts")
+	)
 	(embedded_fonts no)

Commit message: encoder breakout rev a
Parts:
- removed J1: Conn_01x08_MountingPin, Connector_PinSocket_2.54mm:PinSocket_1x08_P2.54mm_Vertical
- removed encoderWithKailh1: ~, encLibrary:EC35AwithKailhSocket
- added ENC1: ~, blitz_lib:EC35A_nosocket, F.Cu at (150.6, 101.0)
- added G***: LOGO, LOGO, F.Cu at (170.2, 84.1)
- added G***: LOGO, LOGO, F.Cu at (132.6, 115.1)
- added J2: Conn_01x07_Pin, Connector_PinHeader_2.54mm:PinHeader_1x07_P2.54mm_Vertical, F.Cu at (142.6, 74.9)
- added REF**: MountingHole_3.2mm_M3_DIN965_Pad_TopBottom, MountingHole:MountingHole_3.2mm_M3_DIN965_Pad_TopBottom, F.Cu at (126.0, 71.6)
- added REF**: MountingHole_3.2mm_M3_DIN965_Pad_TopBottom, MountingHole:MountingHole_3.2mm_M3_DIN965_Pad_TopBottom, F.Cu at (176.0, 71.6)
- added REF**: MountingHole_3.2mm_M3_DIN965_Pad_TopBottom, MountingHole:MountingHole_3.2mm_M3_DIN965_Pad_TopBottom, F.Cu at (176.0, 121.4)
- added REF**: MountingHole_3.2mm_M3_DIN965_Pad_TopBottom, MountingHole:MountingHole_3.2mm_M3_DIN965_Pad_TopBottom, F.Cu at (126.0, 121.4)
- added REV_NEOPIXEL1: ~, blitz_lib:reverse_neopixel, F.Cu at (150.6, 101.0)
- added SOCKET1: ~, blitz_lib:kailh_socket, F.Cu at (150.6, 101.0)
Routing:
- net GND: track 0.00 -> 99.0 mm, vias 0 -> 1
- net /ENC_A: track 0.00 -> 59.9 mm
- net /ENC_B: track 0.00 -> 54.5 mm
- net /NEO_DIN: track 0.00 -> 44.5 mm
- net /NEO_DOUT: track 0.00 -> 39.9 mm
- net +3.3V: track 0.00 -> 35.5 mm
- net /SWITCH: track 0.00 -> 21.5 mm
Other:
- board size 49.5 x 51.5 mm -> 60 x 60 mm
- board text added: "DIN"
- board text added: "DOUT"
- board text added: "ENC_A"
- board text added: "ENC_B"
- board text added: "GND"
- board text added: "Rev A, May 2026"
- board text added: "Rotary Encoder / MX Breakout"
- board text added: "SWITCH"
- board text added: "VIN"
